Commit message: message

File: src/rubot_mecanum_description/urdf/rubot_rp.urdf (robot description, URDF)
Before this commit: robot nexus, 8 links, 7 joints
Links:
- link base_link: mass 10 -> 2
- link lower_left_wheel: mass 0.3844 -> 0.05
- link lower_right_wheel: mass 0.3844 -> 0.05
- link upper_left_wheel: mass 0.3844 -> 0.05
- link upper_right_wheel: mass 0.3844 -> 0.05
